File: sg1000.kicad_pcb (KiCad board)
At the start: 2 copper layers, 150 x 134.7 mm, 72 parts, among them CN1 Conn_01x07_Female, J1 USB-B1HSB6, J2 RCJ-014, J3 RCJ-013, Q1 2n4401, Q1c1 2n3906, SW1 Pause Key, SW2 Power Toggle, U1 SG-1000-Cart, U10 PLCCZ80, U100 74HCT574, U101 74HCT574, U102 74HCT574, U103 AS6C62256-DIP, U11 AS6C62256-DIP, U12 TMS9918A, U13 74LS139, U16 74LS32, U18 74LS257, U2 SG-1000-Expansion, U21 74LS257, U3 SN76489AN, U99 74HCT04, X2 10.73863MHz

Commit message: track cleanup
Other:
- board text added: "d0"
- board text added: "d7"
Changed lines of the file:
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@@
     (property "Sheetfile" "sg1000.kicad_sch")
     (property "Sheetname" "")
-    (fp_text reference "U2" (at 0 -0.5 -90 unlocked) (layer "F.SilkS")
+    (fp_text reference "U2" (at 0 -0.5 -90 unlocked) (layer "F.SilkS") hide
       (effects (font (size 1 1) (thickness 0.15)))
     )
@@
     (effects (font (size 1 1) (thickness 0.15)))
   )
+  (gr_text "d7" (at 159.893 95.758) (layer "F.SilkS")
+    (effects (font (size 1 1) (thickness 0.15)))
+  )
   (gr_text "WRAM_A11" (at 78.232 114.3 90) (layer "F.SilkS")
     (effects (font (size 1 1) (thickness 0.15)))
@@
     (effects (font (size 0.9 0.9) (thickness 0.15)))
   )
+  (gr_text "d0" (at 159.893 113.284) (layer "F.SilkS")
+    (effects (font (size 1 1) (thickness 0.15)))
+  )
   (gr_text "CONTROLLER 1" (at 76.2 179.451) (layer "F.SilkS")
     (effects (font (size 1.5 1.5) (thickness 0.375)) (justify right))
@@
   (via (at 16.383 70.358) (size 0.8) (drill 0.4) (layers "F.Cu" "B.Cu") (net 2))
   (segment (start 62.992 123.317) (end 63.5 123.825) (width 1) (layer "B.Cu") (net 2))
-  (segment (start 16.637 68.58) (end 16.637 69.088) (width 1) (layer "B.Cu") (net 2))
+  (segment (start 16.637 68.58) (end 16.637 70.104) (width 1) (layer "B.Cu") (net 2))
   (segment (start 29.845 72.2175) (end 25.8275 68.2) (width 1) (layer "B.Cu") (net 2))
   (segment (start 113.03 149.833115) (end 113.03 159.893) (width 1) (layer "B.Cu") (net 2))
   (segment (start 60.833 70.485) (end 61.087 70.231) (width 1) (layer "B.Cu") (net 2))
   (segment (start 62.088 148.331) (end 62.088 144.033) (width 1) (layer "B.Cu") (net 2))
-  (segment (start 16.637 69.088) (end 16.637 70.104) (width 1) (layer "B.Cu") (net 2))
   (segment (start 74.803 143.637) (end 74.803 144.302) (width 1) (layer "B.Cu") (net 2))
   (segment (start 84.455 52.07) (end 84.455 55.617) (width 1) (layer "B.Cu") (net 2))

Commit message: Bevel and edge cleanup
Parts:
- moved REF** 0.25 mm to (160.3, 177.3)
Other:
- board size 150 x 134.7 mm -> 149.7 x 134.7 mm
