File: romcart/romcart.kicad_sch (KiCad schematic)
At the start: 4 parts

Commit message: Awful PCB outline
Parts:
- added C1: 0.1µF, Capacitor_THT:C_Disc_D6.0mm_W2.5mm_P5.00mm, symbol Device:C_Small
- JP1: renamed from JP?; footprint (none) -> Jumper:SolderJumper-2_P1.3mm_Bridged_RoundedPad1.0x1.5mm
- U2: renamed from U?; footprint (none) -> SoggyCartridge:CartridgeEdge
- gave numbers to parts that had none: 2
Connections:
- net 5V: now also JP1.2 (B), C1.1
- net GND: now also C1.2; no longer JP1.2 (B)
Other:
- note added: "This pin will be used for cartridge-detect/autoboot on Soggy v3+ - must be connected to 5V for it to work"
- note removed: "This pin is used for cartridge-detect/autoboot on Soggy v3+ - must be connected to ground for it to work"
Changed lines of the file:
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@@
+    (stroke (width 0) (type default) (color 0 0 0 0))
+  )
+  (wire (pts (xy 69.85 104.775) (xy 69.85 105.41))
     (stroke (width 0) (type default) (color 0 0 0 0))
   )
@@
     (stroke (width 0) (type default) (color 0 0 0 0))
   )
-  (wire (pts (xy 164.465 57.785) (xy 168.275 57.785))
-    (stroke (width 0) (type default) (color 0 0 0 0))
-  )
   (wire (pts (xy 86.995 73.025) (xy 89.535 73.025))
     (stroke (width 0) (type default) (color 0 0 0 0))
@@
     (stroke (width 0) (type default) (color 0 0 0 0))
   )
+  (wire (pts (xy 164.465 57.785) (xy 169.545 57.785))
+    (stroke (width 0) (type default) (color 0 0 0 0))
+  )
   (wire (pts (xy 148.59 93.345) (xy 154.305 93.345))
     (stroke (width 0) (type default) (color 0 0 0 0))
@@
     (effects (font (size 1.27 1.27)) (justify left bottom))
   )
-  (text "This pin is used for cartridge-detect/autoboot\non Soggy v3+ - must be connected to ground\nfor it to work"
-    (at 174.625 59.69 0)
+  (text "This pin will be used for cartridge-detect/autoboot\non Soggy v3+ - must be connected to 5V\nfor it to work"
+    (at 173.355 60.96 0)
     (effects (font (size 1.27 1.27)) (justify left bottom))
   )
@@
     (effects (font (size 1.27 1.27)) (justify left bottom))
   )
-  (label "GND" (at 168.275 57.785 0)
-    (effects (font (size 1.27 1.27)) (justify left bottom))
-  )
   (label "A15" (at 112.395 95.885 0)
     (effects (font (size 1.27 1.27)) (justify left bottom))
@@
     (effects (font (size 1.27 1.27)) (justify left bottom))
   )
+  (label "5V" (at 169.545 57.785 0)
+    (effects (font (size 1.27 1.27)) (justify left bottom))
+  )
   (label "D7" (at 86.995 75.565 180)
     (effects (font (size 1.27 1.27)) (justify right bottom))
@@
     (effects (font (size 1.27 1.27)) (justify right bottom))
   )
+  (label "5V" (at 69.85 104.775 90)
+    (effects (font (size 1.27 1.27)) (justify left bottom))
+  )
   (label "~{RD}" (at 112.395 103.505 0)
     (effects (font (size 1.27 1.27)) (justify left bottom))
@@
     (effects (font (size 1.27 1.27)) (justify right bottom))
   )
+  (label "GND" (at 69.85 110.49 270)
+    (effects (font (size 1.27 1.27)) (justify right bottom))
+  )
   (label "D3" (at 124.46 113.665 180)
     (effects (font (size 1.27 1.27)) (justify right bottom))
@@
   (label "5V" (at 120.65 45.085 90)
     (effects (font (size 1.27 1.27)) (justify left bottom))
+  )
+  (symbol (lib_id "Device:C_Small") (at 69.85 107.95 0) (unit 1)
+    (in_bom yes) (on_board yes) (fields_autoplaced)
+    (property "Reference" "C1" (id 0) (at 72.39 106.6862 0)
+      (effects (font (size 1.27 1.27)) (justify left))
+    )
+    (property "Value" "0.1µF" (id 1) (at 72.39 109.2262 0)
+      (effects (font (size 1.27 1.27)) (justify left))
+    )
+    (property "Footprint" "Capacitor_THT:C_Disc_D6.0mm_W2.5mm_P5.00mm" (id 2) (at 69.85 107.95 0)
+      (effects (font (size 1.27 1.27)) hide)
+    )
+    (property "Datasheet" "~" (id 3) (at 69.85 107.95 0)
+      (effects (font (size 1.27 1.27)) hide)
+    )
+    (pin "1")
+    (pin "2")
   )
   (symbol (lib_id "Memory_EPROM:27C512") (at 99.695 80.645 0) (mirror y) (unit 1)
     (in_bom yes) (on_board yes) (fields_autoplaced)
-    (property "Reference" "U?" (id 0) (at 100.2156 49.53 0)
+    (property "Reference" "U1" (id 0) (at 100.2156 49.53 0)
       (effects (font (size 1.27 1.27)) (justify right))
     )
@@
   (symbol (lib_id "LeadedSolder:SG-1000-Cart") (at 135.89 66.675 0) (unit 1)
     (in_bom yes) (on_board yes) (fields_autoplaced)
-    (property "Reference" "U?" (id 0) (at 137.9094 46.99 0)
+    (property "Reference" "U2" (id 0) (at 137.9094 46.99 0)
       (effects (font (size 1.27 1.27)) (justify left))
     )
@@
       (effects (font (size 1.27 1.27)) (justify left))
     )
-    (property "Footprint" "" (id 2) (at 132.08 66.675 0)
+    (property "Footprint" "SoggyCartridge:CartridgeEdge" (id 2) (at 132.08 66.675 0)
       (effects (font (size 1.27 1.27)) hide)
     )
@@
   (symbol (lib_id "Jumper:Jumper_2_Bridged") (at 159.385 57.785 0) (unit 1)
     (in_bom yes) (on_board yes) (fields_autoplaced)
-    (property "Reference" "JP?" (id 0) (at 159.385 54.61 0))
+    (property "Reference" "JP1" (id 0) (at 159.385 54.61 0))
     (property "Value" "Jumper_2_Bridged" (id 1) (at 159.385 54.61 0)
       (effects (font (size 1.27 1.27)) hide)
     )
-    (property "Footprint" "" (id 2) (at 159.385 57.785 0)
+    (property "Footprint" "Jumper:SolderJumper-2_P1.3mm_Bridged_RoundedPad1.0x1.5mm" (id 2) (at 159.385 57.785 0)
       (effects (font (size 1.27 1.27)) hide)
     )
@@
   (symbol (lib_id "Switch:SW_SPDT") (at 114.935 116.84 0) (unit 1)
     (in_bom yes) (on_board yes) (fields_autoplaced)
-    (property "Reference" "SW?" (id 0) (at 114.935 109.22 0))
+    (property "Reference" "SW1" (id 0) (at 114.935 109.22 0))
     (property "Value" "SW_SPDT" (id 1) (at 114.935 111.76 0))
     (property "Footprint" "Connector_PinHeader_2.54mm:PinHeader_1x03_P2.54mm_Vertical" (id 2) (at 114.935 116.84 0)
@@
   )
   (symbol_instances
+    (path "/14d27f4c-87f8-4720-a041-e480665bf6d0"
+      (reference "C1") (unit 1) (value "0.1µF") (footprint "Capacitor_THT:C_Disc_D6.0mm_W2.5mm_P5.00mm")
+    )
     (path "/c5e9e9d8-bb9f-4b46-b198-9fc69b2f3ac4"
-      (reference "JP?") (unit 1) (value "Jumper_2_Bridged") (footprint "")
+      (reference "JP1") (unit 1) (value "Jumper_2_Bridged") (footprint "Jumper:SolderJumper-2_P1.3mm_Bridged_RoundedPad1.0x1.5mm")
     )
     (path "/f5f580bc-325f-40e5-9926-61cdad866883"
-      (reference "SW?") (unit 1) (value "SW_SPDT") (footprint "Connector_PinHeader_2.54mm:PinHeader_1x03_P2.54mm_Vertical")
+      (reference "SW1") (unit 1) (value "SW_SPDT") (footprint "Connector_PinHeader_2.54mm:PinHeader_1x03_P2.54mm_Vertical")
     )
     (path "/2f86a5a7-f5ca-4ab8-9522-155140e227f5"
-      (reference "U?") (unit 1) (value "27C512") (footprint "Socket:DIP_Socket-28_W11.9_W12.7_W15.24_W17.78_W18.5_3M_228-1277-00-0602J")
+      (reference "U1") (unit 1) (value "27C512") (footprint "Socket:DIP_Socket-28_W11.9_W12.7_W15.24_W17.78_W18.5_3M_228-1277-00-0602J")
     )
     (path "/ab3fe2af-889a-4baf-ae59-e1bc253ec9ae"
-      (reference "U?") (unit 1) (value "SG-1000-Cart") (footprint "")
-    )
-  )
+      (reference "U2") (unit 1) (value "SG-1000-Cart") (footprint "SoggyCartridge:CartridgeEdge")
+    )
+  )

Commit message: Route begins
Parts:
- added J1: Proto Connector, Connector_PinSocket_2.54mm:PinSocket_2x22_P2.54mm_Vertical, symbol Connector_Generic:Conn_02x22_Top_Bottom
Connections:
- net 5V: now also J1.23 (Pin_23)
- net CA7: now also J1.36 (Pin_36)
- net D0: now also J1.15 (Pin_15)
- net D1: now also J1.16 (Pin_16)
- net D2: now also J1.17 (Pin_17)
- net D3: now also J1.18 (Pin_18)
- net D4: now also J1.19 (Pin_19)
- net D5: now also J1.20 (Pin_20)
- net D6: now also J1.21 (Pin_21)
- net D7: now also J1.22 (Pin_22)
- net GND: now also J1.43 (Pin_43), J1.44 (Pin_44)
- net ~{CAS0}: now also J1.35 (Pin_35)
- net ~{CAS1}: now also J1.38 (Pin_38)
- net ~{CONT}: now also J1.33 (Pin_33)
- net ~{CSCN4}: now also J1.24 (Pin_24)
- net ~{CSRAM}: now also J1.25 (Pin_25)
- net ~{EXM1}: now also J1.26 (Pin_26)
- net ~{IORD}: now also J1.29 (Pin_29)
- net ~{IOWR}: now also J1.30 (Pin_30)
- net ~{M1}: now also J1.42 (Pin_42)
- net ~{MREQ}: now also J1.32 (Pin_32)
- net ~{RAS0}: now also J1.34 (Pin_34)
- net ~{RAS1}: now also J1.37 (Pin_37)
- net ~{RCSEL}: now also J1.39 (Pin_39)
- net ~{RD}: now also J1.27 (Pin_27)
- net ~{RFSH}: now also J1.31 (Pin_31)
- net ~{WR}: now also J1.28 (Pin_28)
- net A0: now reaches U1.10 (A0), U2.A1 (A0)
- net A0: now also J1.1 (Pin_1)
- net A12: now reaches U1.2 (A12), U2.A13 (A12)
- net A12: now also J1.13 (Pin_13)
- net A10: now reaches U1.21 (A10), U2.A11 (A10)
- net A10: now also J1.11 (Pin_11)
- net A11: now reaches U1.23 (A11), U2.A12 (A11)
- net A11: now also J1.12 (Pin_12)
- net A9: now reaches U1.24 (A9), U2.A10 (A9)
- net A9: now also J1.10 (Pin_10)
- net A8: now reaches U1.25 (A8), U2.A9 (A8)
- net A8: now also J1.9 (Pin_9)
- net A13: now reaches U1.26 (A13), U2.A14 (A13)
- net A13: now also J1.14 (Pin_14)
- net A14: now reaches U1.27 (A14), U2.B18 (A14)
- net A14: now also J1.40 (Pin_40)
- net A7: now reaches U1.3 (A7), U2.A8 (A7)
- net A7: now also J1.8 (Pin_8)
- net A6: now reaches U1.4 (A6), U2.A7 (A6)
- net A6: now also J1.7 (Pin_7)
- net A5: now reaches U1.5 (A5), U2.A6 (A5)
- net A5: now also J1.6 (Pin_6)
- net A4: now reaches U1.6 (A4), U2.A5 (A4)
- net A4: now also J1.5 (Pin_5)
- net A3: now reaches U1.7 (A3), U2.A4 (A3)
- net A3: now also J1.4 (Pin_4)
- net A2: now reaches U1.8 (A2), U2.A3 (A2)
- net A2: now also J1.3 (Pin_3)
- net A1: now reaches U1.9 (A1), U2.A2 (A1)
- net A1: now also J1.2 (Pin_2)
- new net ~{EXM2}: J1.41 (Pin_41)
Other:
- note added: ""A side""
- note added: ""B side""

Commit message: Full route
Connections:
- net ~{EXM2}: now also U1.20 (~{CE}), U2.B19 (~{EXM2})
Changed lines of the file:
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@@
     (effects (font (size 1.27 1.27)) (justify right bottom))
+  )
+  (label "~{EXM2}" (at 112.395 100.965 0)
+    (effects (font (size 1.27 1.27)) (justify left bottom))
   )
   (label "5V" (at 120.65 45.085 90)
