File: romcart/romcart.kicad_pcb (KiCad board)
At the start: 2 copper layers, 72 x 50.2 mm, 5 parts, among them SW1 SW_SPDT, U1 27C512, U2 SG-1000-Cart

Commit message: Route begins
Parts:
- added J1: Proto Connector, Connector_PinSocket_2.54mm:PinSocket_2x22_P2.54mm_Vertical, F.Cu at (126.9, 78.1)
Connections:
- net Net-(U1-Pad10) renamed /A0
- net Net-(U1-Pad2) renamed /A12
- net Net-(U1-Pad21) renamed /A10
- net Net-(U1-Pad23) renamed /A11
- net Net-(U1-Pad24) renamed /A9
- net Net-(U1-Pad25) renamed /A8
- net Net-(U1-Pad26) renamed /A13
- net Net-(U1-Pad27) renamed /A14
- net Net-(U1-Pad3) renamed /A7
- net Net-(U1-Pad4) renamed /A6
- net Net-(U1-Pad5) renamed /A5
- net Net-(U1-Pad6) renamed /A4
- net Net-(U1-Pad7) renamed /A3
- net Net-(U1-Pad8) renamed /A2
- net Net-(U1-Pad9) renamed /A1
- JP1 pad 2: /GND -> /5V
Routing:
- net /GND: track 34.7 -> 26.9 mm
- net /5V: track 27.5 -> 35.3 mm
- added copper zone on F.Cu, net /5V

Commit message: Full route
Connections:
- U1 pad 20: Net-(U1-Pad20) -> /~{EXM2}
- U2 pad B19: Net-(U1-Pad20) -> /~{EXM2}
Routing:
- net /D4: track 0.00 -> 127.0 mm, vias 0 -> 5
- net /D5: track 0.00 -> 126.2 mm, vias 0 -> 5
- net /D3: track 0.00 -> 122.3 mm, vias 0 -> 5
- net /D7: track 0.00 -> 120.1 mm, vias 0 -> 5
- net /D6: track 0.00 -> 118.0 mm, vias 0 -> 5
- net /A6: track 0.00 -> 96.4 mm, vias 0 -> 4
- net /D2: track 0.00 -> 95.4 mm, vias 0 -> 4
- net /~{EXM2}: track 0.00 -> 93.9 mm, vias 0 -> 4
- net /A7: track 0.00 -> 92.6 mm, vias 0 -> 4
- net /D1: track 0.00 -> 88.2 mm, vias 0 -> 4
- net /~{RD}: track 0.00 -> 86.5 mm, vias 0 -> 4
- net /D0: track 0.00 -> 86.0 mm, vias 0 -> 4
- net /~{IORD}: track 0.00 -> 85.8 mm, vias 0 -> 2
- net /A4: track 0.00 -> 85.1 mm, vias 0 -> 4
- net /A5: track 0.00 -> 79.8 mm, vias 0 -> 3
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Other:
- board text added: "5v"
- board text added: "A0"
- board text added: "A1"
- board text added: "A10"
- board text added: "A11"
- board text added: "A12"
- board text added: "A13"
- board text added: "A14"
- board text added: "A2"
- board text added: "A3"
- board text added: "A4"
- board text added: "A5"
- board text added: "A6"
- board text added: "A7"
- board text added: "A8"
- board text added: "A9"
- board text added: "D0"
- board text added: "D1"
- board text added: "D2"
- board text added: "D3"
- board text added: "D4"
- board text added: "D5"
- board text added: "D6"
- board text added: "D7"
- board text added: "GND"
- board text added: "~{CONT}"
- board text added: "~{CSCN4}"
- board text added: "~{EXM1}"
- board text added: "~{EXM2}"
- board text added: "~{IORD}"
- board text added: "~{IOWR}"
- board text added: "~{M1}"
- board text added: "~{MREQ}"
- board text added: "~{RD}"
- board text added: "~{RFSH}"
- board text added: "~{WR}"

Commit message: Logos
Parts:
- added G***: LOGO, Logos:Soggy, F.Cu at (119.4, 101.3)
Routing:
- net /~{RCSEL}: track 56.0 -> 61.9 mm
Other:
- board text added: "A22"
- board text added: "B1"
- board text added: "B22"
- board text added: "BACK"
- board text added: "FRONT"
- board text added: "ROM A15 Switch"
- board text added: "leadedsolder.com 2022"
- board text added: "soggy cartridge v0.1"
- board text removed: "A15 Switch"
