File: keyboard/sg1000.kicad_pcb (KiCad board)
At the start: 2 copper layers, 147 parts, among them J1 USB_B_Micro, J2 Conn_02x03_Odd_Even, K0 KEYSW, K1 KEYSW, K10 KEYSW, K11 KEYSW, K12 KEYSW, K13 KEYSW, K14 KEYSW, K15 KEYSW, K16 KEYSW, K17 KEYSW, K18 KEYSW, K19 KEYSW, K2 KEYSW, K20 KEYSW, K21 KEYSW, K22 KEYSW, K23 KEYSW, K24 KEYSW, K25 KEYSW, K26 KEYSW, K27 KEYSW, K28 KEYSW, K29 KEYSW, K3 KEYSW, K30 KEYSW, K31 KEYSW, K32 KEYSW, K33 KEYSW, K34 KEYSW, K35 KEYSW, K36 KEYSW, K37 KEYSW, K38 KEYSW, K39 KEYSW, K4 KEYSW, K40 KEYSW, K41 KEYSW, K42 KEYSW, K43 KEYSW, K44 KEYSW, K45 KEYSW, K46 KEYSW, K47 KEYSW, K48 KEYSW, K49 KEYSW, K5 KEYSW, K50 KEYSW, K51 KEYSW, K52 KEYSW, K53 KEYSW, K54 KEYSW, K55 KEYSW, K56 KEYSW, K57 KEYSW, K58 KEYSW, K59 KEYSW, K6 KEYSW, K60 KEYSW, K61 KEYSW, K62 KEYSW, K7 KEYSW, K8 KEYSW, K9 KEYSW, SW1 Reset_SW, U1 ATmega32U4-AU, Y1 Crystal

Commit message: Sega header added, not right fp yet
Parts:
- removed C6, C7: 22p, Capacitor_SMD:C_0805_2012Metric_Pad1.15x1.40mm_HandSolder
- removed C8: 1u, Capacitor_SMD:C_0805_2012Metric_Pad1.15x1.40mm_HandSolder
- removed R1, R4: 10k, Resistor_SMD:R_0805_2012Metric_Pad1.15x1.40mm_HandSolder
- removed R2, R3: 22R, Resistor_SMD:R_0805_2012Metric_Pad1.15x1.40mm_HandSolder
- removed SW1: Reset_SW, Button_Switch_SMD:SW_Push_1P1T_NO_6x6mm_H9.5mm
- removed Y1: Crystal, Crystal:Crystal_SMD_5032-2Pin_5.0x3.2mm_HandSoldering
- added JP1: SolderJumper_2_Bridged, Jumper:SolderJumper-2_P1.3mm_Bridged_RoundedPad1.0x1.5mm, F.Cu at (209.9, 22.1)
- J1: value USB_B_Micro -> SEGA BUS; footprint Connector_USB:USB_Micro-B_Wuerth_629105150521_CircularHoles -> Connector_PinHeader_2.54mm:PinHeader_2x25_P2.54mm_Vertical; moved to F.Cu
- U1: value ATmega32U4-AU -> 8255; footprint Package_QFP:TQFP-44_10x10mm_P0.8mm -> Package_DIP:DIP-40_W15.24mm; moved to F.Cu
- moved J1 354.3 mm to (-99.3, 18.3), turned to 90 degrees
- moved U1 128.8 mm to (190.9, 22.4), turned to 0 degrees
Connections:
- net /Col_15 renamed Net-(U1-Pad19)
- net /Col_16 renamed Net-(U1-Pad20)
- net /Col_17 renamed Net-(U1-Pad21)
- net /Row_5 renamed Net-(U1-Pad8)
- net /Row_6 renamed Net-(U1-Pad1)
- J1 pad 2: Net-(J1-Pad2) -> VCC
- J1 pad 3: Net-(J1-Pad3) -> VCC
- J1 pad 4: Net-(J1-Pad4) -> VCC
- J1 pad 5: GND -> Net-(J1-Pad5)
- J1 pad 6: GND -> Net-(J1-Pad6)
- U1 pad 10: /Row_3 -> Net-(U1-Pad10)
- U1 pad 11: /Row_2 -> Net-(U1-Pad11)
- U1 pad 12: /Row_1 -> Net-(U1-Pad12)
- U1 pad 13: /Reset -> Net-(U1-Pad13)
- U1 pad 14: VCC -> Net-(U1-Pad14)
- U1 pad 15: GND -> Net-(U1-Pad15)
- U1 pad 18: /Row_0 -> Net-(U1-Pad18)
- U1 pad 2: VCC -> Net-(U1-Pad2)
- U1 pad 22: /Col_14 -> Net-(U1-Pad22)
- U1 pad 23: GND -> Net-(U1-Pad23)
- U1 pad 24: VCC -> Net-(U1-Pad24)
- U1 pad 25: /Col_7 -> Net-(U1-Pad25)
- U1 pad 26: /Col_6 -> VCC
- U1 pad 27: /Col_5 -> Net-(U1-Pad27)
- U1 pad 28: /Col_4 -> Net-(U1-Pad28)
- U1 pad 29: /Col_3 -> Net-(U1-Pad29)
- U1 pad 30: /Col_2 -> Net-(U1-Pad30)
- U1 pad 31: /Col_1 -> Net-(U1-Pad31)
- U1 pad 32: /Col_0 -> Net-(U1-Pad32)
- U1 pad 34: VCC -> Net-(U1-Pad34)
- U1 pad 35: GND -> Net-(JP1-Pad2)
- U1 pad 36: /Col_8 -> Net-(U1-Pad36)
- U1 pad 37: /Col_9 -> Net-(U1-Pad37)
- U1 pad 38: /Col_10 -> Net-(U1-Pad38)
- U1 pad 39: /Col_11 -> Net-(U1-Pad39)
- U1 pad 40: /Col_12 -> Net-(U1-Pad40)
- U1 pad 5: GND -> Net-(U1-Pad5)
- U1 pad 7: VCC -> GND
- U1 pad 9: /Row_4 -> Net-(U1-Pad9)
Routing:
- net Net-(U1-Pad16): track 15.0 -> 0.00 mm
- net Net-(C7-Pad1): track 0.00 -> 15.0 mm
- net Net-(U1-Pad17): track 14.6 -> 0.00 mm
- net Net-(C6-Pad1): track 0.00 -> 14.6 mm
- net Net-(U1-Pad4): track 13.4 -> 0.00 mm
- net Net-(R2-Pad1): track 0.00 -> 13.4 mm
- net Net-(U1-Pad3): track 12.0 -> 0.00 mm
- net Net-(R3-Pad1): track 0.00 -> 12.0 mm
- net Net-(U1-Pad6): track 6.79 -> 0.00 mm
- net Net-(C8-Pad1): track 0.00 -> 6.79 mm
- net Net-(U1-Pad33): track 3.73 -> 0.00 mm
- net Net-(R4-Pad2): track 0.00 -> 3.73 mm
