File: cartridges/mark-iii-romcart/mark-iii-romcart.kicad_pcb (KiCad board)
At the start: 2 copper layers, 72 x 70.5 mm, 9 parts, among them SW1 SW_SPDT, U1 27C512, U2 SG-1000-Cart

Commit message: Carts to KiCad 7
Other:
- board text added: "Back"
